File: kicad/ardustat.kicad_pcb (KiCad board)
At the start: 2 copper layers, 60 x 56 mm, 12 parts, among them J1 Power, J2 TM1637, J3 Enc, J4 Relay, J5 NTC, Q1 BC547

Commit message: upd
Parts:
- added H1: MountingHole, MountingHole:MountingHole_3.2mm_M3_DIN965_Pad, F.Cu at (27.0, 35.0)
- added H2: MountingHole, MountingHole:MountingHole_3.2mm_M3_DIN965_Pad, F.Cu at (81.0, 35.0)
- added H3: MountingHole, MountingHole:MountingHole_3.2mm_M3_DIN965_Pad, F.Cu at (27.0, 85.0)
- added H4: MountingHole, MountingHole:MountingHole_3.2mm_M3_DIN965_Pad, F.Cu at (81.0, 85.0)
Other:
- board size 60 x 56 mm -> 62 x 58 mm
