File: kicad/ardustat.kicad_sch (KiCad schematic)
At the start: 10 parts, among them J1 Power, J2 TM1637, J3 Enc, J4 Relay, J5 NTC, Q1 BC547

Commit message: upd
Parts:
- added H1, H2, H3, H4: MountingHole, MountingHole:MountingHole_3.2mm_M3_DIN965_Pad, symbol Mechanical:MountingHole
